File: panel/stemcell-panel.kicad_pcb (KiCad board)
At the start: 2 copper layers, 87.6 x 73 mm, 258 parts, among them J1 USB C Connector, J2 Left, J3 Right, J4 Down, SW1 Boot0, U1 STM32F4x1CxUx, U2 XC6220B331MR, Y1 HSE1 8Mhz 12pF

Commit message: Version bump, new renders, 3D models
- v2.0.0 to v2.1.0
- added uncommon 3D models to stemcell footprint library
- re-rendered front and back images.
Other:
- board text added: "v2.1.0"
- board text removed: "v2.0.0"
Changed lines of the file:
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@@
       (svguseinch false)
       (svgprecision 6)
-      (excludeedgelayer true)
+      (excludeedgelayer false)
       (plotframeref false)
       (viasonmask false)
@@
       (drillshape 0)
       (scaleselection 1)
-      (outputdirectory "panel/")
+      (outputdirectory "panel/gerbers/")
     )
   )
@@
     (effects (font (size 0.7 0.7) (thickness 0.08)) (justify mirror))
   )
-  (gr_text "v2.0.0" (at 123.5514 73.92 180) (layer "B.SilkS")
+  (gr_text "v2.1.0" (at 123.5514 73.92 180) (layer "B.SilkS")
     (effects (font (size 0.7 0.7) (thickness 0.1)) (justify mirror))
   )
@@
     (effects (font (size 0.7 0.7) (thickness 0.08)) (justify mirror))
   )
-  (gr_text "v2.0.0" (at 69.4886 56.255) (layer "B.SilkS")
+  (gr_text "v2.1.0" (at 69.4886 56.255) (layer "B.SilkS")
     (effects (font (size 0.7 0.7) (thickness 0.1)) (justify mirror))
   )
@@
     (effects (font (size 0.7 0.7) (thickness 0.08)) (justify mirror))
   )
-  (gr_text "v2.0.0" (at 93.6186 56.255) (layer "B.SilkS")
+  (gr_text "v2.1.0" (at 93.6186 56.255) (layer "B.SilkS")
     (effects (font (size 0.7 0.7) (thickness 0.1)) (justify mirror))
   )
@@
     (effects (font (size 0.7 0.7) (thickness 0.08)) (justify mirror))
   )
-  (gr_text "v2.0.0" (at 117.7486 56.255) (layer "B.SilkS")
+  (gr_text "v2.1.0" (at 117.7486 56.255) (layer "B.SilkS")
     (effects (font (size 0.7 0.7) (thickness 0.1)) (justify mirror))
   )
@@
     (effects (font (size 0.7 0.7) (thickness 0.08)) (justify mirror))
   )
-  (gr_text "v2.0.0" (at 99.4214 73.92 180) (layer "B.SilkS")
+  (gr_text "v2.1.0" (at 99.4214 73.92 180) (layer "B.SilkS")
     (effects (font (size 0.7 0.7) (thickness 0.1)) (justify mirror))
   )
@@
     (effects (font (size 0.7 0.7) (thickness 0.08)) (justify mirror))
   )
-  (gr_text "v2.0.0" (at 75.2914 73.92 180) (layer "B.SilkS")
+  (gr_text "v2.1.0" (at 75.2914 73.92 180) (layer "B.SilkS")
     (effects (font (size 0.7 0.7) (thickness 0.1)) (justify mirror))
   )
